Commit message: URDF 최종근사판(12URDF0725) 교체: 제로샷 통과 — 낙상 0/64, 12kg 정합 1.144
- make_base_urdf.py 신설(§4-1 1단계 자동화): 링크명 통일, base 주입,
  축규약 검사·복원. 익스포트 결함 2건 자동 교정(left_hip_r 관절명 오타,
  left_hip_f 축 반전 — 방치 시 비대칭 리밋 거울반전)
- 질량 9.94→10.49kg(+5.6%), 기구 동일. 게이트: 리밋 12주입·부호 12/12 일치
  (7-19 합격판과 수치 동일)·스폰 개루프 FAIL은 구 자산 동일 거동(회귀 아님)
- 배포정책 model_8997 재학습 없이 통과: 직립 2.75°, 발목롤 4.75<5.0,
  페이로드 그리드 12/13 (앞+5kg만 한계 23% — 배터리 위/뒤 장착 권장)
- stage3 질량 캘리브 1.15~1.26→1.09~1.19, eval 기본 스케일 1.21→1.144

Co-Authored-By: Claude Fable 5 <noreply@anthropic.com>
Claude-Session: https://claude.ai/code/session_01S4YXFodgAK6C1yVTW22JbY

File: rl_walking/assets/biped12_base.urdf (robot description, URDF)
Before this commit: robot biped12, 14 links, 13 joints
Links:
- link left_ankle_f_joint: mass 0.486119247655161 -> 0.4765; geometry collision mesh filename=/home/ryu/humanoid_leg_test1/12URDF0725/meshes/left_ankle_f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; visual mesh filename=/home/ryu/humanoid_leg_test1/12URDF0725/meshes/left_ankle_f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
- link left_ankle_r_joint: mass 0.50489357707771 -> 0.54241; geometry collision mesh filename=/home/ryu/humanoid_leg_test1/12URDF0725/meshes/left_ankle_r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; visual mesh filename=/home/ryu/humanoid_leg_test1/12URDF0725/meshes/left_ankle_r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
- link left_hip_a_joint: mass 0.632623778007109 -> 0.55773; geometry collision mesh filename=/home/ryu/humanoid_leg_test1/12URDF0725/meshes/left_hip_a_L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; visual mesh filename=/home/ryu/humanoid_leg_test1/12URDF0725/meshes/left_hip_a_L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
- link left_hip_f_joint: mass 0.393578984491956 -> 0.39358; geometry collision mesh filename=/home/ryu/humanoid_leg_test1/12URDF0725/meshes/left_hip_f_L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; visual mesh filename=/home/ryu/humanoid_leg_test1/12URDF0725/meshes/left_hip_f_L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
- link left_hip_r_joint: mass 0.581468457020583 -> 0.67544; geometry collision mesh filename=/home/ryu/humanoid_leg_test1/12URDF0725/meshes/left_hip_r_L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; visual mesh filename=/home/ryu/humanoid_leg_test1/12URDF0725/meshes/left_hip_r_L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
- link left_knee_joint: mass 0.602009778953134 -> 0.6077; geometry collision mesh filename=/home/ryu/humanoid_leg_test1/12URDF0725/meshes/left_knee_Li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; visual mesh filename=/home/ryu/humanoid_leg_test1/12URDF0725/meshes/left_knee_Li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
- link pelvis: mass 3.54036668275575 -> 3.9846; geometry collision mesh filename=/home/ryu/humanoid_leg_test1/12URDF0725/meshes/pelvis.STL; visual mesh filename=/home/ryu/humanoid_leg_test1/12URDF0725/meshes/pelvis.STL
- link right_ankle_f_joint: mass 0.48130619869307 -> 0.48131; geometry collision mesh filename=/home/ryu/humanoid_leg_test1/12URDF0725/meshes/right_ankle_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; visual mesh filename=/home/ryu/humanoid_leg_test1/12URDF0725/meshes/right_ankle_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
- link right_ankle_r_joint: mass 0.504893577077711 -> 0.54241; geometry collision mesh filename=/home/ryu/humanoid_leg_test1/12URDF0725/meshes/right_ankle_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; visual mesh filename=/home/ryu/humanoid_leg_test1/12URDF0725/meshes/right_ankle_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
- link right_hip_a_joint: mass 0.632623778007108 -> 0.55181; geometry collision mesh filename=/home/ryu/humanoid_leg_test1/12URDF0725/meshes/right_hip_a_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; visual mesh filename=/home/ryu/humanoid_leg_test1/12URDF0725/meshes/right_hip_a_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
- link right_hip_f_joint: mass 0.393578984491956 -> 0.39358; geometry collision mesh filename=/home/ryu/humanoid_leg_test1/12URDF0725/meshes/right_hip_f_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; visual mesh filename=/home/ryu/humanoid_leg_test1/12URDF0725/meshes/right_hip_f_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
- link right_hip_r_joint: mass 0.581468457020582 -> 0.67544; geometry collision mesh filename=/home/ryu/humanoid_leg_test1/12URDF0725/meshes/right_hip_r_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; visual mesh filename=/home/ryu/humanoid_leg_test1/12URDF0725/meshes/right_hip_r_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
- link right_knee_joint: mass 0.602009778953135 -> 0.6077; geometry collision mesh filename=/home/ryu/humanoid_leg_test1/12URDF0725/meshes/right_knee_L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; visual mesh filename=/home/ryu/humanoid_leg_test1/12URDF0725/meshes/right_knee_L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
Joints:
- joint left_ankle_f_joint: limit lower=0 upper=0 effort=0 velocity=0 -> (none)
- joint left_ankle_r_joint: limit lower=0 upper=0 effort=0 velocity=0 -> (none)
- joint left_hip_a_joint: limit lower=0 upper=0 effort=0 velocity=0 -> (none)
- joint left_hip_f_joint: limit lower=0 upper=0 effort=0 velocity=0 -> (none)
- joint left_hip_r_joint: limit lower=0 upper=0 effort=0 velocity=0 -> (none)
- joint left_knee_joint: limit lower=0 upper=0 effort=0 velocity=0 -> (none); origin xyz=-0.02015 -0.15828 0.00035 rpy=0 0 0 -> xyz=-0.01985 -0.15827 0.00035 rpy=0 0 0
- joint right_hip_a_joint: limit lower=0 upper=0 effort=0 velocity=0 -> (none)
- joint right_hip_f_joint: limit lower=0 upper=0 effort=0 velocity=0 -> (none)
- joint right_knee_joint: origin xyz=0.02015 -0.15828 -0.00035 rpy=0 0 0 -> xyz=0.01985 -0.15827 -0.00035 rpy=0 0 0
