Commit message: final1 자산 수복 완료 — 스폰 즉사 원인은 base↔hip_a 자기충돌 관입, 페어 필터로 치유
증상: final1 자산(패드 유무 무관)으로는 kp150 강체홀드조차 64/64 즉사.
com/imu 주입과 무관하게 낙상 방향까지 동일 → 물리 차이가 아니라 자산 결함.

판별 사슬 (대조군 전부 실측):
- 헐 자산 0단계 오늘 재실행 0/64·+0.0699 → 하네스 무죄
- 패드 제거 변형도 64/64 → 패드 무죄
- 구 URDF 오늘 재변환 0/64·+0.0699(원본과 동일) → 변환 파이프라인 무죄
- 전신 CoM 구/신 동일(전후 -13.5 vs -13.1mm) → 질량 분포 무죄
- 프로브 실측: 스폰 k=0에 base_contact 종료 발화, base 6,443N ·
  좌우 hip_a 각 ~10,000N. base 힘 = -(hip_a 힘 합) → 페어는 base↔hip_a 확정.

원인: 신형 골반 메시가 횡 ±122mm(구 ±87~95)로 커졌고(전장·프로파일 편입),
hip_a도 모터 편입으로 152mm 길어져, self-collision ON(발 자기충돌용)에서
비인접 페어 base↔hip_a 의 콘벡스 근사가 ~28mm 상호관입.
골반 convexDecomposition 만으론 불충분(힘 불변) — hip_a 헐이 자기 오목부를
메우는 것까지는 못 고침.

수복: UsdPhysics.FilteredPairsAPI 로 base↔left/right_hip_a 페어 필터
(rl_walking/scripts/patch_usd_filter_pairs.py, 루트 레이어 over 저작).
정당성: 실물은 설계 공차로 비접촉, 실간섭은 자기충돌 스윕 기반 관절리밋이
이미 차단. 지면↔base/hip_a 접촉(낙상 판정)은 유지됨.
부수: 골반 approximation=convexDecomposition 유지(낙상 시 타페어 정합),
make_base_urdf.py 가 소문자 _link 도 *_joint 로 개명(env 정규식 계약).

수복 후 검증 (log_picture/02f*, 드리프트DR_{H0b,P0b,P2b,P4b}):
- 0·1단계: 0/64, 추세 -0.0149°/s (헐 +0.0699 보다 0에 근접), 에너지 0.237
- v6b 배터리 (deploy old·still, 헐 대비):
    com0   낙상 21.9%→26.6%, 추세 +0.86→+1.01
    comR   낙상 65.6%→70.3%, 추세 +2.18→+2.61
    combo  낙상 84.4%→85.9%, 추세 +3.33→**+4.09 ≈ 실물 +4.06**
- 낙상 방향 반전: 헐은 4방 균등, 패드는 좌/우 지배(P2b 왼18·오른11)
  — 패드 횡폭 ±38mm(헐 ±45) 축소의 직접 증거
- 떨림: E_smth 0.41→0.44~0.48(+8~16%), RMS +9~11% — 실물 4.40 은 여전히
  미재현. 강체 패드 기하만으론 부족 → 잔여 후보 = 패드 고무 컴플라이언스

교훈: 임포터의 병합·근사 콜리전은 링크 구성이 바뀌면 자기충돌 지형이
통째로 바뀐다. 새 자산은 반드시 0단계(강체홀드)부터 태운다.

Co-Authored-By: Claude Fable 5 <noreply@anthropic.com>
Claude-Session: https://claude.ai/code/session_01S4YXFodgAK6C1yVTW22JbY

File: rl_walking/assets/biped12_final1.urdf (robot description, URDF)
Before this commit: robot biped12, 24 links, 23 joints
Links:
- removed link left_ankle_f_link
- removed link left_ankle_r_link
- removed link left_hip_a_link
- removed link left_hip_f_link
- removed link left_hip_r_link
- removed link left_knee_link
- removed link right_ankle_f_link
- removed link right_ankle_r_link
- removed link right_hip_a_link
- removed link right_hip_f_link
- removed link right_hip_r_link
- removed link right_knee_link
- added link left_ankle_f_joint, mass 0.479350778376135; collision mesh filename=/home/ryu/humanoid_leg_test1/final1_urdf/meshes/left_ankle_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; visual mesh filename=/home/ryu/humanoid_leg_test1/final1_urdf/meshes/left_ankle_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
- added link left_ankle_r_joint, mass 0.552773293782394; collision mesh filename=/home/ryu/humanoid_leg_test1/final1_urdf/meshes/left_ankle_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; visual mesh filename=/home/ryu/humanoid_leg_test1/final1_urdf/meshes/left_ankle_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
- added link left_hip_a_joint, mass 0.7989; collision mesh filename=/home/ryu/humanoid_leg_test1/final1_urdf/meshes/left_hip_a_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; visual mesh filename=/home/ryu/humanoid_leg_test1/final1_urdf/meshes/left_hip_a_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
- added link left_hip_f_joint, mass 0.3995; collision mesh filename=/home/ryu/humanoid_leg_test1/final1_urdf/meshes/left_hip_f_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; visual mesh filename=/home/ryu/humanoid_leg_test1/final1_urdf/meshes/left_hip_f_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
- added link left_hip_r_joint, mass 0.48458; collision mesh filename=/home/ryu/humanoid_leg_test1/final1_urdf/meshes/left_hip_r_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; visual mesh filename=/home/ryu/humanoid_leg_test1/final1_urdf/meshes/left_hip_r_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
- added link left_knee_joint, mass 0.6077; collision mesh filename=/home/ryu/humanoid_leg_test1/final1_urdf/meshes/left_knee_l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; visual mesh filename=/home/ryu/humanoid_leg_test1/final1_urdf/meshes/left_knee_l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
- added link right_ankle_f_joint, mass 0.479350778376136; collision mesh filename=/home/ryu/humanoid_leg_test1/final1_urdf/meshes/right_ankle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; visual mesh filename=/home/ryu/humanoid_leg_test1/final1_urdf/meshes/right_ankle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
- added link right_ankle_r_joint, mass 0.55277329273497; collision mesh filename=/home/ryu/humanoid_leg_test1/final1_urdf/meshes/right_ankle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; visual mesh filename=/home/ryu/humanoid_leg_test1/final1_urdf/meshes/right_ankle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
- added link right_hip_a_joint, mass 0.75198145394561; collision mesh filename=/home/ryu/humanoid_leg_test1/final1_urdf/meshes/right_hip_a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; visual mesh filename=/home/ryu/humanoid_leg_test1/final1_urdf/meshes/right_hip_a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
- added link right_hip_f_joint, mass 0.399500067678193; collision mesh filename=/home/ryu/humanoid_leg_test1/final1_urdf/meshes/right_hip_f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; visual mesh filename=/home/ryu/humanoid_leg_test1/final1_urdf/meshes/right_hip_f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
- added link right_hip_r_joint, mass 0.484578164755911; collision mesh filename=/home/ryu/humanoid_leg_test1/final1_urdf/meshes/right_hip_r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; visual mesh filename=/home/ryu/humanoid_leg_test1/final1_urdf/meshes/right_hip_r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
- added link right_knee_joint, mass 0.607696213986947; collision mesh filename=/home/ryu/humanoid_leg_test1/final1_urdf/meshes/right_knee_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; visual mesh filename=/home/ryu/humanoid_leg_test1/final1_urdf/meshes/right_knee_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
Joints:
- joint left_ankle_f_joint: child left_ankle_f_link -> left_ankle_f_joint; parent left_knee_link -> left_knee_joint
- joint left_ankle_r_joint: child left_ankle_r_link -> left_ankle_r_joint; parent left_ankle_f_link -> left_ankle_f_joint
- joint left_hip_a_joint: child left_hip_a_link -> left_hip_a_joint; parent left_hip_f_link -> left_hip_f_joint
- joint left_hip_f_joint: child left_hip_f_link -> left_hip_f_joint
- joint left_hip_r_joint: child left_hip_r_link -> left_hip_r_joint; parent left_hip_a_link -> left_hip_a_joint
- joint left_knee_joint: child left_knee_link -> left_knee_joint; parent left_hip_r_link -> left_hip_r_joint
- joint leftfoot_leftback_RA30P: parent left_ankle_r_link -> left_ankle_r_joint
- joint leftfoot_leftfront_RA30P: parent left_ankle_r_link -> left_ankle_r_joint
- joint leftfoot_rightback_RA30P: parent left_ankle_r_link -> left_ankle_r_joint
- joint leftfoot_rightfront_RA30P: parent left_ankle_r_link -> left_ankle_r_joint
- joint right_ankle_f_joint: child right_ankle_f_link -> right_ankle_f_joint; parent right_knee_link -> right_knee_joint
- joint right_ankle_r_joint: child right_ankle_r_link -> right_ankle_r_joint; parent right_ankle_f_link -> right_ankle_f_joint
- joint right_hip_a_joint: child right_hip_a_link -> right_hip_a_joint; parent right_hip_f_link -> right_hip_f_joint
- joint right_hip_f_joint: child right_hip_f_link -> right_hip_f_joint
- joint right_hip_r_joint: child right_hip_r_link -> right_hip_r_joint; parent right_hip_a_link -> right_hip_a_joint
- joint right_knee_joint: child right_knee_link -> right_knee_joint; parent right_hip_r_link -> right_hip_r_joint
- joint rightfoot_leftfback_RA30P: parent right_ankle_r_link -> right_ankle_r_joint
- joint rightfoot_leftfront_RA30P: parent right_ankle_r_link -> right_ankle_r_joint
- joint rightfoot_rightfback_RA30P: parent right_ankle_r_link -> right_ankle_r_joint
- joint rightfoot_rightfront_RA30P: parent right_ankle_r_link -> right_ankle_r_joint
