Commit message: 정정: hip_r PLA 변형 URDF 의 대체 범위 — 링크 전체가 아니라 회전 모터(611 g)+원통 하우징(288 g)
무엇: biped12_final3_hiprpla.urdf 를 다시 만들었다. 앞 판(83342580)은 hip_r 링크 전체(모터~무릎 클램프 258 mm)를 211 g 으로 바꿨는데, 실제 출력물은 회전 모터와 그 하우징만 대체하고 무릎 쪽은 그대로다(사용자가 그림에 표시해 확인, 무게는 실측). 하우징은 URDF 에서 hip_a 링크 아랫부분이라 hip_a(0.967 → 0.891)·hip_r(0.936 → 0.325) 두 링크를 고쳤다. 전체 17.635 → 16.260 kg.
왜 틀렸나: hip_r 링크 메시가 무릎 클램프까지 이어진 한 덩어리라 '모터+하우징 = 링크 전체'로 읽었다. 부품 경계를 사용자에게 그림으로 확인받기 전에 값을 넣은 것이 잘못.
검증: 생성 스크립트가 새 관성의 양정치·삼각 부등식을 확인. 평가기가 실행 중 읽은 네 링크 질량·질량 중심·관성이 URDF 와 일치(전체 16.2595 kg). 정정판 평가 7 건 유효(무외란 1/619, 앞 40 N 56.6 %, 앞 램프 23.2 %) — 판정 불변(서기 합격·밀기 불합격).
미검증: 뒤 18 N(고정 변위 0.325° 로 무효 2 회), seed 1–2 개뿐, 원통 근사의 오차, 공중 시작·걷기. 평가는 사용자 지시로 중단.
가설로만 남김: 잘못 잡은 범위(−0.725 kg/쪽)와 정정판(−0.688 kg/쪽)의 앞 밀기 낙상이 같은 급 → 빠지는 위치보다 양이 지배적(seed 1 개).

Co-Authored-By: Claude Opus 5.5 <noreply@anthropic.com>
Claude-Session: https://claude.ai/code/session_016BSW7xbbyGTjJtK7yX5Y1U

File: rl_walking/assets/biped12_final3_hiprpla.urdf (robot description, URDF)
Before this commit: robot biped12, 24 links, 23 joints
Links:
- link left_hip_a_joint: mass 0.96740276 -> 0.89063276
- link left_hip_r_joint: mass 0.21123 -> 0.32534972
- link right_hip_a_joint: mass 0.96740276 -> 0.89063276
- link right_hip_r_joint: mass 0.21123 -> 0.32534972
