Commit message: 저장소 정리 — URDF 소스 한곳(urdf/), 구 파생자산 archive/, 모델 레지스트리(models/)·세대 보고서(reports/) 신설, 리포트 월별 정리
삭제 없음, 전부 이동(git mv):
- urdf/{URDF12DOF, 12URDF0725, final1_urdf, final2_urdf(첫 커밋), final3_urdf} + README(계보·익스포터 고질병)
- rl_walking/assets/archive/{biped12_final1, usd_final1, footvar, symbox, payload} + README
- 파생 URDF 4종·isaacsim_scene 메시 절대경로, make_base_urdf/fix_final1_frames/fix_final3_mesh 경로, .gitignore 갱신
- log_picture/{2026-07, 2026-08}/ (mtime 기준), 0904_무효_버그창/ (eval_drift_dr _rl 섀도잉 창 산출물 + 이분탐색·분리실험, README)
- reports/audits/ (02f/02g/02h 자산·하네스 감사), reports/gen_v14~v17 (gen_report.py 자동 생성), reports/README(세대 대조표·판정 기준),
  reports/audit_0905_adversarial.json (100 에이전트 감사 결과: 확정 31/기각 0)
- models/{stand_v14,v14s,v15,v16,v17} + legacy/{v6b,v7,v13}: policy.pt/onnx·env/agent.yaml·meta.json(md5) — logs/ 가 gitignore 라 재현 단위를 버전관리
- docs/INDEX.md; 신규 도구 gen_report.py, register_model.py
근거: 10.49kg 자산(URDF 정합 낮음) 세대와 17.62kg 실질량 세대를 구조로 분리하라는 승윤님 지시(0905).

Co-Authored-By: Claude Fable 5.1 <noreply@anthropic.com>
Claude-Session: https://claude.ai/code/session_01S4YXFodgAK6C1yVTW22JbY

File: isaacsim_scene/newURDF12DOF_isaac.urdf (robot description, URDF)
Before this commit: robot newURDF12DOF, 13 links, 12 joints
Links:
- link left_ankle_f_joint: geometry collision mesh filename=/home/ryu/humanoid_leg_test1/urdf/URDF12DOF/meshes/left_ank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; visual mesh filename=/home/ryu/humanoid_leg_test1/urdf/URDF12DOF/meshes/left_ank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
- link left_ankle_r_joint: geometry collision mesh filename=/home/ryu/humanoid_leg_test1/urdf/URDF12DOF/meshes/left_ank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; visual mesh filename=/home/ryu/humanoid_leg_test1/urdf/URDF12DOF/meshes/left_ank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
- link left_hip_a_joint: geometry collision mesh filename=/home/ryu/humanoid_leg_test1/urdf/URDF12DOF/meshes/left_hip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; visual mesh filename=/home/ryu/humanoid_leg_test1/urdf/URDF12DOF/meshes/left_hip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
- link left_hip_f_joint: geometry collision mesh filename=/home/ryu/humanoid_leg_test1/urdf/URDF12DOF/meshes/left_hip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; visual mesh filename=/home/ryu/humanoid_leg_test1/urdf/URDF12DOF/meshes/left_hip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
- link left_hip_r_joint: geometry collision mesh filename=/home/ryu/humanoid_leg_test1/urdf/URDF12DOF/meshes/left_hip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; visual mesh filename=/home/ryu/humanoid_leg_test1/urdf/URDF12DOF/meshes/left_hip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
- link left_knee_joint: geometry collision mesh filename=/home/ryu/humanoid_leg_test1/urdf/URDF12DOF/meshes/left_kne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; visual mesh filename=/home/ryu/humanoid_leg_test1/urdf/URDF12DOF/meshes/left_kne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
- link pelvis: geometry collision mesh filename=/home/ryu/humanoid_leg_test1/urdf/URDF12DOF/meshes/pelvis.S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; visual mesh filename=/home/ryu/humanoid_leg_test1/urdf/URDF12DOF/meshes/pelvis.S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
- link right_ankle_f_joint: geometry collision mesh filename=/home/ryu/humanoid_leg_test1/urdf/URDF12DOF/meshes/right_an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; visual mesh filename=/home/ryu/humanoid_leg_test1/urdf/URDF12DOF/meshes/right_an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
- link right_ankle_r_joint: geometry collision mesh filename=/home/ryu/humanoid_leg_test1/urdf/URDF12DOF/meshes/right_an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; visual mesh filename=/home/ryu/humanoid_leg_test1/urdf/URDF12DOF/meshes/right_an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
- link right_hip_a_joint: geometry collision mesh filename=/home/ryu/humanoid_leg_test1/urdf/URDF12DOF/meshes/right_hi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; visual mesh filename=/home/ryu/humanoid_leg_test1/urdf/URDF12DOF/meshes/right_hi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
- link right_hip_f_joint: geometry collision mesh filename=/home/ryu/humanoid_leg_test1/urdf/URDF12DOF/meshes/right_hi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; visual mesh filename=/home/ryu/humanoid_leg_test1/urdf/URDF12DOF/meshes/right_hi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
- link right_hip_r_joint: geometry collision mesh filename=/home/ryu/humanoid_leg_test1/urdf/URDF12DOF/meshes/right_hi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; visual mesh filename=/home/ryu/humanoid_leg_test1/urdf/URDF12DOF/meshes/right_hi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
- link right_knee_joint: geometry collision mesh filename=/home/ryu/humanoid_leg_test1/urdf/URDF12DOF/meshes/right_kn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; visual mesh filename=/home/ryu/humanoid_leg_test1/urdf/URDF12DOF/meshes/right_kn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

File: rl_walking/assets/biped12_base.urdf (robot description, URDF)
Before this commit: robot biped12, 14 links, 13 joints
Links:
- link left_ankle_f_joint: geometry collision mesh filename=/home/ryu/humanoid_leg_test1/urdf/12URDF0725/meshes/left_an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; visual mesh filename=/home/ryu/humanoid_leg_test1/urdf/12URDF0725/meshes/left_an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
- link left_ankle_r_joint: geometry collision mesh filename=/home/ryu/humanoid_leg_test1/urdf/12URDF0725/meshes/left_an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; visual mesh filename=/home/ryu/humanoid_leg_test1/urdf/12URDF0725/meshes/left_an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
- link left_hip_a_joint: geometry collision mesh filename=/home/ryu/humanoid_leg_test1/urdf/12URDF0725/meshes/left_hi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; visual mesh filename=/home/ryu/humanoid_leg_test1/urdf/12URDF0725/meshes/left_hi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
- link left_hip_f_joint: geometry collision mesh filename=/home/ryu/humanoid_leg_test1/urdf/12URDF0725/meshes/left_hi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; visual mesh filename=/home/ryu/humanoid_leg_test1/urdf/12URDF0725/meshes/left_hi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
- link left_hip_r_joint: geometry collision mesh filename=/home/ryu/humanoid_leg_test1/urdf/12URDF0725/meshes/left_hi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; visual mesh filename=/home/ryu/humanoid_leg_test1/urdf/12URDF0725/meshes/left_hi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
- link left_knee_joint: geometry collision mesh filename=/home/ryu/humanoid_leg_test1/urdf/12URDF0725/meshes/left_kn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; visual mesh filename=/home/ryu/humanoid_leg_test1/urdf/12URDF0725/meshes/left_kn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
- link pelvis: geometry collision mesh filename=/home/ryu/humanoid_leg_test1/urdf/12URDF0725/meshes/pelvis.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; visual mesh filename=/home/ryu/humanoid_leg_test1/urdf/12URDF0725/meshes/pelvis.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
- link right_ankle_f_joint: geometry collision mesh filename=/home/ryu/humanoid_leg_test1/urdf/12URDF0725/meshes/right_a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; visual mesh filename=/home/ryu/humanoid_leg_test1/urdf/12URDF0725/meshes/right_a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
- link right_ankle_r_joint: geometry collision mesh filename=/home/ryu/humanoid_leg_test1/urdf/12URDF0725/meshes/right_a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; visual mesh filename=/home/ryu/humanoid_leg_test1/urdf/12URDF0725/meshes/right_a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
- link right_hip_a_joint: geometry collision mesh filename=/home/ryu/humanoid_leg_test1/urdf/12URDF0725/meshes/right_h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; visual mesh filename=/home/ryu/humanoid_leg_test1/urdf/12URDF0725/meshes/right_h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
- link right_hip_f_joint: geometry collision mesh filename=/home/ryu/humanoid_leg_test1/urdf/12URDF0725/meshes/right_h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; visual mesh filename=/home/ryu/humanoid_leg_test1/urdf/12URDF0725/meshes/right_h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
- link right_hip_r_joint: geometry collision mesh filename=/home/ryu/humanoid_leg_test1/urdf/12URDF0725/meshes/right_h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; visual mesh filename=/home/ryu/humanoid_leg_test1/urdf/12URDF0725/meshes/right_h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
- link right_knee_joint: geometry collision mesh filename=/home/ryu/humanoid_leg_test1/urdf/12URDF0725/meshes/right_k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; visual mesh filename=/home/ryu/humanoid_leg_test1/urdf/12URDF0725/meshes/right_k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

File: rl_walking/assets/biped12_final3.urdf (robot description, URDF)
Before this commit: robot biped12, 24 links, 23 joints
Links:
- link D455: geometry collision mesh filename=/home/ryu/humanoid_leg_test1/urdf/final3_urdf/meshes/D455.S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; visual mesh filename=/home/ryu/humanoid_leg_test1/urdf/final3_urdf/meshes/D455.S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
- link imu: geometry collision mesh filename=/home/ryu/humanoid_leg_test1/urdf/final3_urdf/meshes/imu.STL; visual mesh filename=/home/ryu/humanoid_leg_test1/urdf/final3_urdf/meshes/imu.STL
- link left_ankle_f_joint: geometry collision mesh filename=/home/ryu/humanoid_leg_test1/urdf/final3_urdf/meshes/left_a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; visual mesh filename=/home/ryu/humanoid_leg_test1/urdf/final3_urdf/meshes/left_a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
- link left_ankle_r_joint: geometry collision mesh filename=/home/ryu/humanoid_leg_test1/urdf/final3_urdf/meshes/left_a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; visual mesh filename=/home/ryu/humanoid_leg_test1/urdf/final3_urdf/meshes/left_a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
- link left_hip_a_joint: geometry collision mesh filename=/home/ryu/humanoid_leg_test1/urdf/final3_urdf/meshes/left_h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; visual mesh filename=/home/ryu/humanoid_leg_test1/urdf/final3_urdf/meshes/left_h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
- link left_hip_f_joint: geometry collision mesh filename=/home/ryu/humanoid_leg_test1/urdf/final3_urdf/meshes/left_h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; visual mesh filename=/home/ryu/humanoid_leg_test1/urdf/final3_urdf/meshes/left_h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
- link left_hip_r_joint: geometry collision mesh filename=/home/ryu/humanoid_leg_test1/urdf/final3_urdf/meshes/left_h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; visual mesh filename=/home/ryu/humanoid_leg_test1/urdf/final3_urdf/meshes/left_h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
- link left_knee_joint: geometry collision mesh filename=/home/ryu/humanoid_leg_test1/urdf/final3_urdf/meshes/left_k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; visual mesh filename=/home/ryu/humanoid_leg_test1/urdf/final3_urdf/meshes/left_k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
- link leftfoot_leftback_RA30P: geometry collision mesh filename=/home/ryu/humanoid_leg_test1/urdf/final3_urdf/meshes/leftfo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; visual mesh filename=/home/ryu/humanoid_leg_test1/urdf/final3_urdf/meshes/leftfo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
- link leftfoot_leftfront_RA30P: geometry collision mesh filename=/home/ryu/humanoid_leg_test1/urdf/final3_urdf/meshes/leftfo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; visual mesh filename=/home/ryu/humanoid_leg_test1/urdf/final3_urdf/meshes/leftfo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
- link leftfoot_rightback_RA30P: geometry collision mesh filename=/home/ryu/humanoid_leg_test1/urdf/final3_urdf/meshes/leftfo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; visual mesh filename=/home/ryu/humanoid_leg_test1/urdf/final3_urdf/meshes/leftfo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
- link leftfoot_rightfront_RA30P: geometry collision mesh filename=/home/ryu/humanoid_leg_test1/urdf/final3_urdf/meshes/leftfo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; visual mesh filename=/home/ryu/humanoid_leg_test1/urdf/final3_urdf/meshes/leftfo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
- link pelvis: geometry collision mesh filename=/home/ryu/humanoid_leg_test1/urdf/final3_urdf/meshes/pelvis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; visual mesh filename=/home/ryu/humanoid_leg_test1/urdf/final3_urdf/meshes/pelvis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
- link right_ankle_f_joint: geometry collision mesh filename=/home/ryu/humanoid_leg_test1/urdf/final3_urdf/meshes/right_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; visual mesh filename=/home/ryu/humanoid_leg_test1/urdf/final3_urdf/meshes/right_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
- link right_ankle_r_joint: geometry collision mesh filename=/home/ryu/humanoid_leg_test1/urdf/final3_urdf/meshes/right_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; visual mesh filename=/home/ryu/humanoid_leg_test1/urdf/final3_urdf/meshes/right_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
- link right_hip_a_joint: geometry collision mesh filename=/home/ryu/humanoid_leg_test1/urdf/final3_urdf/meshes/right_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; visual mesh filename=/home/ryu/humanoid_leg_test1/urdf/final3_urdf/meshes/right_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
- link right_hip_f_joint: geometry collision mesh filename=/home/ryu/humanoid_leg_test1/urdf/final3_urdf/meshes/right_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; visual mesh filename=/home/ryu/humanoid_leg_test1/urdf/final3_urdf/meshes/right_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
- link right_hip_r_joint: geometry collision mesh filename=/home/ryu/humanoid_leg_test1/urdf/final3_urdf/meshes/right_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; visual mesh filename=/home/ryu/humanoid_leg_test1/urdf/final3_urdf/meshes/right_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
- link right_knee_joint: geometry collision mesh filename=/home/ryu/humanoid_leg_test1/urdf/final3_urdf/meshes/right_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; visual mesh filename=/home/ryu/humanoid_leg_test1/urdf/final3_urdf/meshes/right_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
- link rightfoot_leftfback_RA30P: geometry collision mesh filename=/home/ryu/humanoid_leg_test1/urdf/final3_urdf/meshes/rightf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; visual mesh filename=/home/ryu/humanoid_leg_test1/urdf/final3_urdf/meshes/rightf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
- link rightfoot_leftfront_RA30P: geometry collision mesh filename=/home/ryu/humanoid_leg_test1/urdf/final3_urdf/meshes/rightf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; visual mesh filename=/home/ryu/humanoid_leg_test1/urdf/final3_urdf/meshes/rightf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
- link rightfoot_rightfback_RA30P: geometry collision mesh filename=/home/ryu/humanoid_leg_test1/urdf/final3_urdf/meshes/rightf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; visual mesh filename=/home/ryu/humanoid_leg_test1/urdf/final3_urdf/meshes/rightf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
- link rightfoot_rightfront_RA30P: geometry collision mesh filename=/home/ryu/humanoid_leg_test1/urdf/final3_urdf/meshes/rightf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; visual mesh filename=/home/ryu/humanoid_leg_test1/urdf/final3_urdf/meshes/rightf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

File: rl_walking/assets/biped12_final3f.urdf (robot description, URDF)
Before this commit: robot biped12, 24 links, 23 joints
Links:
- link D455: geometry collision mesh filename=/home/ryu/humanoid_leg_test1/urdf/final3_urdf/meshes/D455.S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; visual mesh filename=/home/ryu/humanoid_leg_test1/urdf/final3_urdf/meshes/D455.S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
- link imu: geometry collision mesh filename=/home/ryu/humanoid_leg_test1/urdf/final3_urdf/meshes/imu.STL; visual mesh filename=/home/ryu/humanoid_leg_test1/urdf/final3_urdf/meshes/imu.STL
- link left_ankle_f_joint: geometry collision mesh filename=/home/ryu/humanoid_leg_test1/urdf/final3_urdf/meshes/left_a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; visual mesh filename=/home/ryu/humanoid_leg_test1/urdf/final3_urdf/meshes/left_a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
- link left_ankle_r_joint: geometry collision mesh filename=/home/ryu/humanoid_leg_test1/urdf/final3_urdf/meshes/left_a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; visual mesh filename=/home/ryu/humanoid_leg_test1/urdf/final3_urdf/meshes/left_a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
- link left_hip_a_joint: geometry collision mesh filename=/home/ryu/humanoid_leg_test1/urdf/final3_urdf/meshes/left_h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; visual mesh filename=/home/ryu/humanoid_leg_test1/urdf/final3_urdf/meshes/left_h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
- link left_hip_f_joint: geometry collision mesh filename=/home/ryu/humanoid_leg_test1/urdf/final3_urdf/meshes/left_h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; visual mesh filename=/home/ryu/humanoid_leg_test1/urdf/final3_urdf/meshes/left_h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
- link left_hip_r_joint: geometry collision mesh filename=/home/ryu/humanoid_leg_test1/urdf/final3_urdf/meshes/left_h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; visual mesh filename=/home/ryu/humanoid_leg_test1/urdf/final3_urdf/meshes/left_h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
- link left_knee_joint: geometry collision mesh filename=/home/ryu/humanoid_leg_test1/urdf/final3_urdf/meshes/left_k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; visual mesh filename=/home/ryu/humanoid_leg_test1/urdf/final3_urdf/meshes/left_k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
- link leftfoot_leftback_RA30P: geometry collision mesh filename=/home/ryu/humanoid_leg_test1/urdf/final3_urdf/meshes/leftfo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; visual mesh filename=/home/ryu/humanoid_leg_test1/urdf/final3_urdf/meshes/leftfo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
- link leftfoot_leftfront_RA30P: geometry collision mesh filename=/home/ryu/humanoid_leg_test1/urdf/final3_urdf/meshes/leftfo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; visual mesh filename=/home/ryu/humanoid_leg_test1/urdf/final3_urdf/meshes/leftfo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
- link leftfoot_rightback_RA30P: geometry collision mesh filename=/home/ryu/humanoid_leg_test1/urdf/final3_urdf/meshes/leftfo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; visual mesh filename=/home/ryu/humanoid_leg_test1/urdf/final3_urdf/meshes/leftfo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
- link leftfoot_rightfront_RA30P: geometry collision mesh filename=/home/ryu/humanoid_leg_test1/urdf/final3_urdf/meshes/leftfo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; visual mesh filename=/home/ryu/humanoid_leg_test1/urdf/final3_urdf/meshes/leftfo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
- link pelvis: geometry collision mesh filename=/home/ryu/humanoid_leg_test1/urdf/final3_urdf/meshes/pelvis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; visual mesh filename=/home/ryu/humanoid_leg_test1/urdf/final3_urdf/meshes/pelvis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
- link right_ankle_f_joint: geometry collision mesh filename=/home/ryu/humanoid_leg_test1/urdf/final3_urdf/meshes/right_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; visual mesh filename=/home/ryu/humanoid_leg_test1/urdf/final3_urdf/meshes/right_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
- link right_ankle_r_joint: geometry collision mesh filename=/home/ryu/humanoid_leg_test1/urdf/final3_urdf/meshes/right_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; visual mesh filename=/home/ryu/humanoid_leg_test1/urdf/final3_urdf/meshes/right_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
- link right_hip_a_joint: geometry collision mesh filename=/home/ryu/humanoid_leg_test1/urdf/final3_urdf/meshes/right_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; visual mesh filename=/home/ryu/humanoid_leg_test1/urdf/final3_urdf/meshes/right_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
- link right_hip_f_joint: geometry collision mesh filename=/home/ryu/humanoid_leg_test1/urdf/final3_urdf/meshes/right_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; visual mesh filename=/home/ryu/humanoid_leg_test1/urdf/final3_urdf/meshes/right_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
- link right_hip_r_joint: geometry collision mesh filename=/home/ryu/humanoid_leg_test1/urdf/final3_urdf/meshes/right_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; visual mesh filename=/home/ryu/humanoid_leg_test1/urdf/final3_urdf/meshes/right_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
- link right_knee_joint: geometry collision mesh filename=/home/ryu/humanoid_leg_test1/urdf/final3_urdf/meshes/right_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; visual mesh filename=/home/ryu/humanoid_leg_test1/urdf/final3_urdf/meshes/right_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
- link rightfoot_leftfback_RA30P: geometry collision mesh filename=/home/ryu/humanoid_leg_test1/urdf/final3_urdf/meshes/rightf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; visual mesh filename=/home/ryu/humanoid_leg_test1/urdf/final3_urdf/meshes/rightf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
- link rightfoot_leftfront_RA30P: geometry collision mesh filename=/home/ryu/humanoid_leg_test1/urdf/final3_urdf/meshes/rightf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; visual mesh filename=/home/ryu/humanoid_leg_test1/urdf/final3_urdf/meshes/rightf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
- link rightfoot_rightfback_RA30P: geometry collision mesh filename=/home/ryu/humanoid_leg_test1/urdf/final3_urdf/meshes/rightf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; visual mesh filename=/home/ryu/humanoid_leg_test1/urdf/final3_urdf/meshes/rightf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
- link rightfoot_rightfront_RA30P: geometry collision mesh filename=/home/ryu/humanoid_leg_test1/urdf/final3_urdf/meshes/rightf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; visual mesh filename=/home/ryu/humanoid_leg_test1/urdf/final3_urdf/meshes/rightf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
